Commit message: Update launch files to set model type to nav_car and adjust URDF file path; refine common macros for accurate wheel positioning

File: nav_car_description/urdf/include/common_macros.urdf.xacro (robot description, xacro)
@@ -335,6 +335,6 @@
       <child link="base_link" />
       <!-- origin xyz="0 0 ${wheel_radius - base_z_origin_to_wheel_origin}" rpy="0 0 0" /-->
-      <!-- origin xyz="0 0 ${wheel_props['wheel']['radius'] - wheel_props['wheel']['z_offset'] + 0.1}" rpy="0 0 0" /-->
-      <origin xyz="0 0 0" rpy="0 0 0" />
+      <origin xyz="0 0 ${wheel_props['wheel']['radius'] - wheel_props['wheel']['z_offset']}" rpy="0 0 0" />
+      <!-- <origin xyz="0 0 0" rpy="0 0 0" /> -->
     </joint>
   </xacro:macro>

File: nav_car_description/urdf/nav_car.urdf.xacro (robot description, xacro)
@@ -13,4 +13,6 @@
   <xacro:property name="motor_yaml" value="$(find ${package_name})/config/${robot_name}/motor.yaml" />
   <xacro:property name="motor_props" value="${xacro.load_yaml(motor_yaml)}"/>
+  <!-- Footprint link -->
+  <xacro:footprint wheel_props="${back_wheel_props}" />
   <!-- Base link -->
   <xacro:base base_prop="${base_props}" >
