Commit message: Add laser sensor configuration and integration in URDF files

File: nav_car_description/urdf/include/common_sensors.xacro (robot description, xacro)
@@ -64,3 +64,246 @@
   </gazebo>
 </xacro:macro>
+<xacro:macro name="laser" params="prefix parent_link sensor_prop enable_gpu:=true">
+  <xacro:property name="mesh"
+     value="${sensor_prop['laser']['mesh']}"/>
+  <xacro:if value="${enable_gpu}">
+    <xacro:property name="plugin_name" value="libgazebo_ros_gpu_laser.so"/>
+    <xacro:property name="laser_type" value="gpu_ray"/>
+  </xacro:if>
+  <xacro:if value="${not enable_gpu}">
+    <xacro:property name="plugin_name" value="libgazebo_ros_laser.so"/>
+    <xacro:property name="laser_type" value="ray"/>
+  </xacro:if>
+  <link name="${prefix}_laser_link">
+    <xacro:if value="${mesh != '' }" >
+    <visual>
+      <origin xyz="0 0 0" rpy="0 0 ${pi}"/>
+      <geometry>
+        <mesh filename="package://${package_name}/meshes/sensors/${mesh}" />
+      </geometry>
+      <material name="dark_grey"/>
+    </visual>
+  </xacro:if>
+  <xacro:if value="${mesh == '' }" >
+    <visual>
+      <origin xyz="0 0 0" rpy="0 0 0"/>
+        <geometry>
+        <cylinder radius="${sensor_prop['laser']['radius']}" length="${sensor_prop['laser']['length']}"/>
+      </geometry>
+      <material name="red"/>
+    </visual>
+  </xacro:if>
+    <collision>
+      <origin xyz="0 0 0" rpy="0 0 0"/>
+      <geometry>
+        <cylinder radius="${sensor_prop['laser']['radius']}" length="${sensor_prop['laser']['length']}"/>
+      </geometry>
+    </collision>
+    <xacro:cylinder_inertia m="${sensor_prop['laser']['mass']}"
+                            r="${sensor_prop['laser']['radius']}"
+                            l="${sensor_prop['laser']['length']}"
+                            o_xyz="0 0 0"
+                            o_rpy="0 0 0" />
+  </link>
+  <gazebo reference="${prefix}_laser_link">
+    <material>${sensor_prop['laser']['color']}</material>
+  </gazebo>
+  <joint name="${prefix}_laser_joint" type="fixed">
+    <parent link="${parent_link}"/>
+    <child link="${prefix}_laser_link"/>
+    <origin xyz="${sensor_prop['laser']['dx']} ${sensor_prop['laser']['dy']} ${sensor_prop['laser']['dz']}" rpy="0 0 ${pi}"/>
+    <axis xyz="0 1 0" />
+  </joint>
+  <!-- hokuyo gazebo references -->
+  <gazebo reference="${prefix}_laser_link">
+    <!-- type is either gpu_laser or laser -->
+    <sensor type="${laser_type}" name="head_hokuyo_sensor">
+      <pose>0 0 0 0 0 0</pose>
+      <visualize>true</visualize>
+      <update_rate>12</update_rate>
+      <ray>
+        <scan>
+          <horizontal>
+            <samples>360</samples>
+            <resolution>1</resolution>
+            <min_angle>${sensor_prop['laser']['angular_range']['min']}</min_angle>
+            <max_angle>${sensor_prop['laser']['angular_range']['max']}</max_angle>
+          </horizontal>
+        </scan>
+        <range>
+          <min>0.12</min>
+          <max>12.0</max>
+          <resolution>0.01</resolution>
+        </range>
+        <noise>
+          <type>gaussian</type>
+          <!--Noise parameters based on published spec for Hokuyo laser
+               achieving "+-30mm" accuracy at range < 10m.  A mean of 0.0m and
+               stddev of 0.01m will put 99.7% of samples within 0.03m of the true
+               reading. -->
+          <mean>0.0</mean>
+          <stddev>0.01</stddev>
+        </noise>
+      </ray>
+      <!-- plugin_name is either libgazebo_ros_laser.so or libgazebo_ros_gpu_laser.so-->
+      <plugin name="gazebo_ros_head_hokuyo_controller" filename="${plugin_name}">
+        <topicName>/diffbot/scan</topicName>
+        <frameName>${prefix}_laser_link</frameName>
+      </plugin>
+    </sensor>
+  </gazebo>
+</xacro:macro>
+<xacro:macro name="camera_sensor" params=" *joint_origin parent_link sensor_prop visualize mesh:='' ">
+  <link name="camera_link">
+    <xacro:if value="${mesh != '' }" >
+      <visual>
+        <origin xyz="0 0 0" rpy="0 0 0"/>
+        <geometry>
+          <mesh filename="package://${package_name}/meshes/sensors/${mesh}" scale="${sensor_prop['camera']['meshes']['scale']}" />
+        </geometry>
+        <material name="dark_grey"/>
+      </visual>
+    </xacro:if>
+    <xacro:if value="${mesh == '' }" >
+      <visual>
+        <origin xyz="0 0 0" rpy="0 0 0"/>
+        <geometry>
+          <cylinder radius="${sensor_prop['camera']['radius']}" length="${sensor_prop['camera']['length']}"/>
+        </geometry>
+        <material name="red"/>
+      </visual>
+    </xacro:if>
+    <collision>
+      <origin xyz="0 0 0" rpy="0 0 0"/>
+      <geometry>
+        <cylinder radius="0.03" length="0.03"/>
+      </geometry>
+    </collision>
+    <xacro:cylinder_inertia m="${sensor_prop['camera']['mass']}"
+                            r="${sensor_prop['camera']['radius']}"
+                            l="${sensor_prop['camera']['length']}"
+                            o_xyz="0 0 0"
+                            o_rpy="0 0 0" />
+  </link>
+  <gazebo reference="camera_link">
+    <material>Gazebo/Red</material>
+  </gazebo>
+  <joint name="camera_joint" type="fixed">
+    <axis xyz="0 1 0" />
+    <xacro:insert_block name="joint_origin" />
+    <parent link="${parent_link}"/>
+    <child link="camera_link"/>
+  </joint>
+  <gazebo reference="camera_link">
+    <sensor type="camera" name="camera1">
+      <update_rate>60</update_rate>
+      <visualize>${visualize}</visualize>
+      <camera>
+        <horizontal_fov>1.92</horizontal_fov>
+        <image>
+          <width>640</width>
+          <height>480</height>
+          <format>B8G8R8</format>
+        </image>
+        <depth_camera>
+        </depth_camera>
+        <clip>
+          <near>0.02</near>
+          <far>300</far>
+        </clip>
+        <noise>
+          <type>gaussian</type>
+          <!-- Noise is sampled independently per pixel on each frame.
+                That pixel's noise value is added to each of its color
+                channels, which at that point lie in the range [0,1]. -->
+          <mean>0.0</mean>
+          <stddev>0.007</stddev>
+        </noise>
+      </camera>
+      <plugin name="camera_controller" filename="libgazebo_ros_camera.so">
+        <alwaysOn>true</alwaysOn>
+        <updateRate>0.0</updateRate>
+        <cameraName>diffbot/camera1</cameraName>
+        <imageTopicName>image_raw</imageTopicName>
+        <cameraInfoTopicName>camera_info</cameraInfoTopicName>
+        <frameName>camera_link</frameName>
+        <hackBaseline>0.07</hackBaseline>
+        <distortionK1>0.0</distortionK1>
+        <distortionK2>0.0</distortionK2>
+        <distortionK3>0.0</distortionK3>
+        <distortionT1>0.0</distortionT1>
+        <distortionT2>0.0</distortionT2>
+      </plugin>
+    </sensor>
+  </gazebo>
+</xacro:macro>
+<xacro:macro name="imu_sensor" params=" *joint_origin parent_link sensor_prop">
+  <xacro:property name="mesh"
+     value="${sensor_prop['imu']['mesh']}"/>
+  <link name="imu_link">
+    <xacro:if value="${mesh != '' }" >
+      <visual>
+        <origin xyz="0 0 0" rpy="0 0 0"/>
+        <geometry>
+          <mesh filename="package://${package_name}/meshes/sensors/${mesh}" scale="${sensor_prop['imu']['scale']}" />
+        </geometry>
+        <material name="dark_grey"/>
+      </visual>
+    </xacro:if>
+    <xacro:if value="${mesh == '' }" >
+      <visual>
+        <origin xyz="0 0 0" rpy="0 0 0"/>
+        <geometry>
+          <cylinder radius="${sensor_prop['imu']['radius']}" length="${sensor_prop['imu']['length']}"/>
+        </geometry>
+        <material name="red"/>
+      </visual>
+    </xacro:if>
+    <collision>
+      <origin xyz="0 0 0" rpy="0 0 0"/>
+      <geometry>
+        <box size="0.01 0.01 0.01"/>
+      </geometry>
+    </collision>
+    <xacro:box_inertia m="${sensor_prop['imu']['mass']}"
+                       x="${sensor_prop['imu']['size']['x']}"
+                       y="${sensor_prop['imu']['size']['y']}"
+                       z="${sensor_prop['imu']['size']['y']}" />
+    <!-- Todo delete visual>
+      <origin xyz="0 0 0" rpy="0 0 0"/>
+      <geometry>
+        <box size="0.01 0.01 0.01"/>
+      </geometry>
+    </visual>
+    <inertial>
+      <mass value="1e-5" />
+      <origin xyz="0 0 0" rpy="0 0 0"/>
+      <inertia ixx="1e-6" ixy="0" ixz="0" iyy="1e-6" iyz="0" izz="1e-6" />
+    </inertial-->
+  </link>
+  <gazebo reference="imu_link">
+    <material>Gazebo/Yellow</material>
+  </gazebo>
+  <joint name="imu_joint" type="fixed">
+    <axis xyz="0 1 0" />
+    <xacro:insert_block name="joint_origin" />
+    <parent link="${parent_link}"/>
+    <child link="imu_link"/>
+  </joint>
+  <gazebo reference="imu_link">
+    <sensor type="imu" name="my_imu">
+    <always_on>true</always_on>
+    <!-- Publish at 30 hz -->
+    <update_rate>30</update_rate>
+    <plugin name="my_imu_plugin" filename="libgazebo_ros_imu_sensor.so">
+      <ros>
+        <!-- Will publish to /imu/data -->
+        <namespace>/imu</namespace>
+        <argument>~/out:=data</argument>
+      </ros>
+      <!-- frame_name ommited, will be "my_link" -->
+    </plugin>
+    </sensor>
+  </gazebo>
+</xacro:macro>
 </robot>

File: nav_car_description/urdf/nav_car.urdf.xacro (robot description, xacro)
@@ -4,4 +4,5 @@
   <xacro:property name="robot_name" value="nav_car"/>
   <xacro:include filename="$(find ${package_name})/urdf/include/common_macros.urdf.xacro" />
+  <xacro:include filename="$(find ${package_name})/urdf/include/common_sensors.xacro" />
   <!-- <xacro:set_package_name /> -->
   <xacro:property name="back_wheel_yaml" value="$(find ${package_name})/config/${robot_name}/back_wheel.yaml" />
@@ -13,4 +14,6 @@
   <xacro:property name="motor_yaml" value="$(find ${package_name})/config/${robot_name}/motor.yaml" />
   <xacro:property name="motor_props" value="${xacro.load_yaml(motor_yaml)}"/>
+  <xacro:property name="sensor_yaml" value="$(find ${package_name})/config/${robot_name}/sensors.yaml" />
+  <xacro:property name="sensor_prop" value="${xacro.load_yaml(sensor_yaml)}"/>
   <!-- Footprint link -->
   <xacro:footprint wheel_props="${back_wheel_props}" />
@@ -37,4 +40,9 @@
                       base_props="${base_props}" >
   </xacro:motor>
+  <!-- Sensors -->
+  <xacro:laser prefix="lslidar" parent_link="base_link"
+                   sensor_prop="${sensor_prop}"
+                   enable_gpu="${sensor_prop['laser']['enable_gpu']}">
+  </xacro:laser>
   <!-- Front Wheels -->
   <xacro:caster_wheel prefix="rear" reflect="-1"
