Commit message: rename configuration files for nav_car including wheel and base specifications

File: nav_car_description/urdf/nav_car.urdf.xacro (robot description, xacro)
@@ -1,6 +1,6 @@
 <?xml version="1.0"?>
-<robot xmlns:xacro="http://www.ros.org/wiki/xacro" name="nar_car">
-  <xacro:property name="package_name" value="nar_car_description"/>
-  <xacro:property name="robot_name" value="nar_car"/>
+<robot xmlns:xacro="http://www.ros.org/wiki/xacro" name="nav_car">
+  <xacro:property name="package_name" value="nav_car_description"/>
+  <xacro:property name="robot_name" value="nav_car"/>
   <xacro:include filename="$(find ${package_name})/urdf/include/common_macros.urdf.xacro" />
   <!-- <xacro:set_package_name /> -->
@@ -28,4 +28,4 @@
                       wheel_props="${front_wheel_props}">
   </xacro:caster_wheel>
-  <!-- <xacro:include filename="$(find nav_car_description)/urdf/nar_car_gazebo_plugins.xacro"/>  -->
+  <!-- <xacro:include filename="$(find nav_car_description)/urdf/nav_car_gazebo_plugins.xacro"/>  -->
 </robot>

Commit message: fix nav_car configuration for motor control and launch integration

File: nav_car_description/urdf/nav_car.urdf.xacro (robot description, xacro)
@@ -6,9 +6,11 @@
   <!-- <xacro:set_package_name /> -->
   <xacro:property name="back_wheel_yaml" value="$(find ${package_name})/config/${robot_name}/back_wheel.yaml" />
-  <xacro:property name="back_wheel_props" value="${load_yaml(back_wheel_yaml)}"/>
+  <xacro:property name="back_wheel_props" value="${xacro.load_yaml(back_wheel_yaml)}"/>
   <xacro:property name="front_wheel_yaml" value="$(find ${package_name})/config/${robot_name}/front_wheel.yaml" />
-  <xacro:property name="front_wheel_props" value="${load_yaml(front_wheel_yaml)}"/>
+  <xacro:property name="front_wheel_props" value="${xacro.load_yaml(front_wheel_yaml)}"/>
   <xacro:property name="base_yaml" value="$(find ${package_name})/config/${robot_name}/base.yaml" />
-  <xacro:property name="base_props" value="${load_yaml(base_yaml)}"/>
+  <xacro:property name="base_props" value="${xacro.load_yaml(base_yaml)}"/>
+  <xacro:property name="motor_yaml" value="$(find ${package_name})/config/${robot_name}/motor.yaml" />
+  <xacro:property name="motor_props" value="${xacro.load_yaml(motor_yaml)}"/>
   <!-- Base link -->
   <xacro:base base_prop="${base_props}" >
@@ -24,4 +26,13 @@
                       base_props="${base_props}">
   </xacro:wheel>
+  <!-- Motors -->
+  <xacro:motor prefix="back_right" reflect="-1"
+                      motor_props="${motor_props}"
+                      base_props="${base_props}" >
+  </xacro:motor>
+  <xacro:motor prefix="back_left" reflect="1"
+                      motor_props="${motor_props}"
+                      base_props="${base_props}" >
+  </xacro:motor>
   <!-- Front Wheels -->
   <xacro:caster_wheel prefix="rear" reflect="-1"

Commit message: Add IMU joint origin definition and integrate IMU sensor in URDF

File: nav_car_description/urdf/nav_car.urdf.xacro (robot description, xacro)
@@ -16,4 +16,8 @@
   <xacro:property name="sensor_yaml" value="$(find ${package_name})/config/${robot_name}/sensors.yaml" />
   <xacro:property name="sensor_prop" value="${xacro.load_yaml(sensor_yaml)}"/>
+  <!-- 定义 joint_origin -->
+  <xacro:property name="imu_joint_origin">
+    <origin xyz="0 0 0.1" rpy="0 0 0"/>
+  </xacro:property>
   <!-- Footprint link -->
   <xacro:footprint wheel_props="${back_wheel_props}" />
@@ -45,4 +49,6 @@
                    enable_gpu="${sensor_prop['laser']['enable_gpu']}">
   </xacro:laser>
+  <!-- 调用 imu_sensor 宏 -->
+  <xacro:imu_sensor joint_origin="${imu_joint_origin}" parent_link="base_link" sensor_prop="${sensor_prop}" />
   <!-- Front Wheels -->
   <xacro:caster_wheel prefix="rear" reflect="-1"

Commit message: Update tracking frame and trajectory builder parameters for improved performance

File: nav_car_description/urdf/nav_car.urdf.xacro (robot description, xacro)
@@ -49,6 +49,8 @@
                    enable_gpu="${sensor_prop['laser']['enable_gpu']}">
   </xacro:laser>
-  <!-- 调用 imu_sensor 宏 -->
-  <xacro:imu_sensor joint_origin="${imu_joint_origin}" parent_link="base_link" sensor_prop="${sensor_prop}" />
+  <!-- 正确调用 imu_sensor 宏 -->
+  <!-- <xacro:imu_sensor parent_link="base_link" sensor_prop="${sensor_prop}">
+    <origin xyz="0 0 0.1" rpy="0 0 0"/>
+  </xacro:imu_sensor> -->
   <!-- Front Wheels -->
   <xacro:caster_wheel prefix="rear" reflect="-1"
