Commit message: Refactor launch files and configurations for NavCar robot; add extra joints to joint_state_broadcaster, improve TCP server shutdown handling, and update RViz configuration.

File: navcar_description/urdf/nav_car.urdf.xacro (robot description, xacro)
@@ -4,5 +4,5 @@
   <xacro:arg name="use_ros2_control" default="false" />
   <xacro:arg name="use_mock_hardware" default="true" />
-  <xacro:property name="package_name" value="nav_car_description"/>
+  <xacro:property name="package_name" value="navcar_description"/>
   <xacro:property name="robot_name" value="nav_car"/>
   <xacro:include filename="$(find ${package_name})/urdf/include/common_macros.urdf.xacro" />
