Commit message: Fix laser joint origin orientation: set roll, pitch, and yaw to zero for correct alignment.

File: src/navcar_description/urdf/include/common_sensors.xacro (robot description, xacro)
@@ -112,5 +112,5 @@
     <parent link="${parent_link}"/>
     <child link="${prefix}_laser_link"/>
-    <origin xyz="${sensor_prop['laser']['dx']} ${sensor_prop['laser']['dy']} ${sensor_prop['laser']['dz']}" rpy="0 0 ${pi}"/>
+    <origin xyz="${sensor_prop['laser']['dx']} ${sensor_prop['laser']['dy']} ${sensor_prop['laser']['dz']}" rpy="0 0 0"/>
     <axis xyz="0 1 0" />
   </joint>
